File: tiny_schematic/tinyLight.brd (EAGLE design)
At the start: 52 x 33.2 mm, 38 parts, among them IC1 NCP1117, IC2 XMEGA-A4TQFP, IC3 CM1293A-02SR, J1 RASM722PX, J2 Molex, J3 PDI, Q1 BC849SMD, Q2 BC849SMD, X1 MICRO-USB

Commit message: final board (hopefully...)
Parts:
- removed U$9: (no value), ohw-logo:OSHW_8X100_NOTEXT
- added U$1: (no value), ohw-logox:OSHW_8X100_NOTEXT
- SV1: value (none) -> RF/BT
- SV2: value (none) -> UART
- SV3: value (none) -> IR
- moved SV1 2.86 mm to (32.8, 4.90), turned to 0 degrees
- moved R4 2.42 mm to (17.6, 32.1)
- moved C3 1.43 mm to (41.5, 6.90), turned to 90 degrees
- moved J2 1.30 mm to (23.3, 30.1)
- moved C7 0.60 mm to (24.1, 22.5)
- moved R6 0.10 mm to (19.1, 23.2)
Connections:
- removed net N$9: IC2.10, SV1.4
- new net N$1: IC2.10, SV1.3
- net N$8: now also SV1.4; no longer SV1.3
Routing:
- net N$9: track 25.9 -> 0.00 mm
- net N$1: track 0.00 -> 16.2 mm
- net N$8: track 19.9 -> 5.94 mm
- net N$4: track 5.67 -> 17.6 mm
- net +3V3: track 93.4 -> 100.7 mm
- net N$7: track 10.8 -> 17.8 mm
- net N$5: track 12.1 -> 5.99 mm
- net GND: track 225.3 -> 229.1 mm
- net N$6: track 6.44 -> 9.28 mm
- net N$3: track 8.59 -> 10.2 mm
- net I_LUX: track 11.1 -> 12.4 mm
- net PWR_SW: track 46.0 -> 46.5 mm

Commit message: added revision reference, RF net names, fixed cap value
Parts:
- C2: value 110µF -> 10µF
Connections:
- net N$1 renamed CE
- net N$4 renamed SCK
- net N$5 renamed MOSI
- net N$6 renamed MISO
- net N$7 renamed IRQ
- net N$8 renamed CSN
Other:
- board text added: "v1.0"
Changed lines of the file:
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@@
 <rectangle x1="12.5" y1="0.1" x2="27.4" y2="2.9" layer="1"/>
 <rectangle x1="27.6" y1="2.3" x2="42.6" y2="31.3" layer="204"/>
+<text x="46" y="0.9" size="1.778" layer="1">v1.0</text>
 </plain>
 <attributes>
@@
 <element name="R11" library="rcl" package="M2012" value="1k" x="44.4" y="13.8" rot="R180"/>
 <element name="C1" library="rcl" package="C2012" value="10µF" x="19.5" y="8.9" rot="R90"/>
-<element name="C2" library="rcl" package="C2012" value="110µF" x="19.5" y="5.1" rot="R270"/>
+<element name="C2" library="rcl" package="C2012" value="10µF" x="19.5" y="5.1" rot="R270"/>
 <element name="R9" library="rcl" package="M2012" value="150" x="48.4" y="11.2" rot="R180"/>
 <element name="C3" library="rcl" package="C2012" value="100nF" x="41.5" y="6.9" rot="R90"/>
@@
 <wire x1="32.134115625" y1="24.965884375" x2="32.134115625" y2="23.62409375" width="0.4064" layer="1"/>
 </signal>
-<signal name="N$5">
+<signal name="MOSI">
 <contactref element="IC2" pad="15"/>
 <contactref element="SV1" pad="6"/>
@@
 <wire x1="33.734115625" y1="6.505884375" x2="34.07" y2="6.17" width="0.3048" layer="1"/>
 </signal>
-<signal name="N$6">
+<signal name="MISO">
 <contactref element="IC2" pad="16"/>
 <contactref element="SV1" pad="7"/>
@@
 <wire x1="36.61" y1="4.19" x2="36.61" y2="3.63" width="0.3048" layer="1"/>
 </signal>
-<signal name="N$4">
+<signal name="SCK">
 <contactref element="SV1" pad="5"/>
 <contactref element="IC2" pad="17"/>
@@
 <wire x1="34.1" y1="3.8" x2="34.07" y2="3.63" width="0.4064" layer="1"/>
 </signal>
-<signal name="N$7">
+<signal name="IRQ">
 <contactref element="IC2" pad="14"/>
 <contactref element="SV1" pad="8"/>
@@
 <wire x1="33.5" y1="4.9" x2="32.8" y2="5.6" width="0.3048" layer="1"/>
 </signal>
-<signal name="N$8">
+<signal name="CSN">
 <contactref element="IC2" pad="12"/>
 <contactref element="SV1" pad="4"/>
@@
 <wire x1="42.3" y1="22.86" x2="43.3" y2="23.86" width="0.254" layer="1"/>
 </signal>
-<signal name="N$1">
+<signal name="CE">
 <contactref element="IC2" pad="10"/>
 <contactref element="SV1" pad="3"/>

Commit message: fixed colorswirl, added settings preset, minor improvements
Parts:
- SV1: value RF/BT -> RF
Changed lines of the file:
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@@
 <element name="S1" library="tinyLight" package="LSH_6X6" value="SPST_PB" x="48.4" y="27.5" rot="R270"/>
 <element name="C9" library="rcl" package="C2012" value="100nF" x="20.55" y="14.3"/>
-<element name="SV1" library="con-lstb" package="MA04-2" value="RF/BT" x="32.8" y="4.9">
+<element name="SV1" library="con-lstb" package="MA04-2" value="RF" x="32.8" y="4.9">
 <attribute name="OC_NEWARK" value="unknown" x="32.8" y="4.9" size="1.778" layer="27" display="off"/>
 <attribute name="MPN" value="" x="32.8" y="4.9" size="1.778" layer="27" display="off"/>
