File: tiny_schematic/tinyLight.sch (EAGLE design)
At the start: 37 parts, among them IC1 NCP1117, IC2 XMEGA-A4TQFP, IC3 CM1293A-02SR, J1 RASM722PX, J2 Molex, J3 PDI, Q1 BC849SMD, Q2 BC849SMD, X1 MICRO-USB

Commit message: Added comments to schematic; created pdf board documentation
Other:
- note added: "*switched via µC pull-up"
- note added: "Fabian Fritzer & Martin Knapp"
- note added: "GPIO / UART <reserved>"
- note added: "IR receiver"
- note added: "USB power/host detect"
- note added: "input voltage sense (+ lowpass)"
- note added: "led current sensor"
- note added: "led power switch"
- note added: "light sensor"
- note added: "lowpass filter"
- note added: "mode switch"
- note added: "programming / debug interface"
- note added: "solder pad (pin header)"
- note added: "status LED"
- note added: "wireless: NRF24 / BT"
- moved on the sheet: C1, C2, C3, C4, C5, C6, C7, C8, C9, IC1, IC2, IC3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
