File: tiny_schematic/tinyLight_v1.1.brd (EAGLE design)
At the start: 52 x 33.2 mm, 39 parts, among them IC1 NCP1117, IC2 XMEGA-A4TQFP, IC3 CM1293A-02SR, J1 RASM722PX, J2 Molex, J3 PDI, Q1 BC849SMD, Q2 BC849SMD, X1 MICRO-USB

Commit message: Working WS281x implementation (ToDo: Regression Tests)
Parts:
- R6: value 1.5k -> 5.6k
Changed lines of the file:
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@@
 <element name="C8" library="rcl" package="C2012" value="100nF" x="45.9" y="20.3" rot="R90"/>
 <element name="R4" library="rcl" package="M2012" value="5.6k" x="17.6" y="32.1"/>
-<element name="R6" library="rcl" package="M2012" value="1.5k" x="19.1" y="23.2" rot="R180"/>
+<element name="R6" library="rcl" package="M2012" value="5.6k" x="19.1" y="23.2" rot="R180"/>
 <element name="C7" library="rcl" package="C2012" value="100nF" x="24.1" y="22.5" rot="R90"/>
 <element name="S1" library="tinyLight" package="LSH_6X6" value="SPST_PB" x="48.4" y="27.5" rot="R270"/>
